File: placa2.brd (EAGLE design)
At the start: 100 x 81.3 mm, 9 parts

Commit message: feito
Parts:
- added R2, R3, R4, R5, R6: 1K, SparkFun-Resistors:AXIAL-0.3
- moved U$1 4.58 mm to (26.7, 53.3)
- moved R1 1.27 mm to (14.0, 66.0)
Connections:
- new net N$14: J3.2, R6.P$1
- new net N$16: J3.1, R2.P$1
- new net N$21: R3.P$2, U$1.2
- new net N$24: R4.P$2, U$1.1
- net N$3: now also R4.P$1; no longer U$1.1
- net N$5: now also J2.3, R3.P$1; no longer J2.2, U$1.2
- net N$6: now also J3.3, R5.P$1; no longer J2.3, U$1.3
- net N$7: now also R2.P$2; no longer J3.1
- net N$8: now also R6.P$2; no longer J3.2
- net N$9: now also R5.P$2; no longer J3.3
Routing:
- net N$13: track 116.7 -> 64.3 mm
- net N$21: track 0.00 -> 18.1 mm
- net N$4: track 96.9 -> 113.8 mm
- net N$14: track 0.00 -> 15.4 mm
- net N$9: track 24.1 -> 13.0 mm
- net N$24: track 0.00 -> 11.0 mm
- net N$15: track 30.9 -> 41.7 mm
- net N$16: track 0.00 -> 10.3 mm
- net N$5: track 16.4 -> 9.80 mm
- net N$3: track 15.4 -> 9.23 mm
- net N$8: track 21.8 -> 15.8 mm
- net N$6: track 17.5 -> 21.3 mm
- net N$17: track 66.5 -> 63.3 mm
- net N$19: track 35.6 -> 32.8 mm
- net N$10: track 66.2 -> 63.3 mm
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